Commit message: added working seneka_quanjo branch

File: ur_description/urdf/ur10.urdf.xacro (robot description, xacro)
@@ -72,5 +72,11 @@
   <property name="joint_limit_effort" value="300.0" />
   <property name="joint_limit_velocity" value="${pi}" />
-  <xacro:macro name="ur10_robot" params="prefix">
+  <xacro:macro name="ur10_robot" params="prefix parent x y z roll pitch yaw">
+  <!-- Added connector joint for connecting it with a robot -->
+  <joint name="${prefix}ur10_connector" type="fixed">
+    <parent link="${parent}" />
+    <child link = "${prefix}base_link" />
+    <origin xyz="${x} ${y} ${z}" rpy="${roll} ${pitch} ${yaw}" />
+  </joint>
   <link name="${prefix}base_link" >
     <visual>
@@ -87,5 +93,5 @@
     </collision>
     <inertial>
-      <mass value="${base_mass}" />
+      <mass value="${base_mass}"/>
       <inertia ixx="1.0" ixy="0.0" ixz="0.0" iyy="1.0" iyz="0.0" izz="1.0"/>
     </inertial>
@@ -301,8 +307,32 @@
     </inertial>
   </link>
+  <joint name="${prefix}hook_fixed_joint" type="fixed">
+    <parent link="${prefix}wrist_3_link" />
+    <child link = "${prefix}hook_link" />
+    <origin xyz="0.0 ${wrist_3_length} 0.0" rpy="0.0 0.0 ${pi/2.0}" />
+  </joint>
+  <link name="${prefix}hook_link">
+    <visual>
+      <geometry>
+        <mesh filename="package://seneka_ugv_description/meshes/gripper.dae" scale="0.001 0.001 0.001"/>
+      </geometry>
+      <origin xyz="0.0 0.0 0.0" rpy="0.0 -1.57 0.0" />
+    </visual>
+    <collision>
+      <geometry>
+          <mesh filename="package://seneka_ugv_description/meshes/gripper.dae" scale="0.001 0.001 0.001"/>
+      </geometry>
+      <origin xyz="0.0 0.0 0.0" rpy="0.0 -1.57 0.0" />
+    </collision>
+    <inertial>
+      <mass value="1" />
+      <origin xyz="0.0 0.0 0.0" rpy="0.0 0.0 0.0" />
+      <inertia ixx="1.0" ixy="0.0" ixz="0.0" iyy="1.0" iyz="0.0" izz="1.0"/>
+    </inertial>
+  </link>
   <joint name="${prefix}ee_fixed_joint" type="fixed">
-    <parent link="${prefix}wrist_3_link" />
+    <parent link="${prefix}hook_link" />
     <child link = "${prefix}ee_link" />
-    <origin xyz="0.0 ${wrist_3_length} 0.0" rpy="0.0 0.0 ${pi/2.0}" />
+    <origin xyz="0.0 -0.25 0.0" rpy="0.0 0.0 0.0" />
   </joint>
   <link name="${prefix}ee_link" />

Commit message: some beautify changes

File: ur_description/urdf/ur10.urdf.xacro (robot description, xacro)
@@ -72,11 +72,5 @@
   <property name="joint_limit_effort" value="300.0" />
   <property name="joint_limit_velocity" value="${pi}" />
-  <xacro:macro name="ur10_robot" params="prefix parent x y z roll pitch yaw">
-  <!-- Added connector joint for connecting it with a robot -->
-  <joint name="${prefix}ur10_connector" type="fixed">
-    <parent link="${parent}" />
-    <child link = "${prefix}base_link" />
-    <origin xyz="${x} ${y} ${z}" rpy="${roll} ${pitch} ${yaw}" />
-  </joint>
+  <xacro:macro name="ur10_robot" params="prefix">
   <link name="${prefix}base_link" >
     <visual>
@@ -307,32 +301,8 @@
     </inertial>
   </link>
-  <joint name="${prefix}hook_fixed_joint" type="fixed">
+  <joint name="${prefix}ee_fixed_joint" type="fixed">
     <parent link="${prefix}wrist_3_link" />
-    <child link = "${prefix}hook_link" />
+    <child link = "${prefix}ee_link" />
     <origin xyz="0.0 ${wrist_3_length} 0.0" rpy="0.0 0.0 ${pi/2.0}" />
-  </joint>
-  <link name="${prefix}hook_link">
-    <visual>
-      <geometry>
-        <mesh filename="package://seneka_ugv_description/meshes/gripper.dae" scale="0.001 0.001 0.001"/>
-      </geometry>
-      <origin xyz="0.0 0.0 0.0" rpy="0.0 -1.57 0.0" />
-    </visual>
-    <collision>
-      <geometry>
-          <mesh filename="package://seneka_ugv_description/meshes/gripper.dae" scale="0.001 0.001 0.001"/>
-      </geometry>
-      <origin xyz="0.0 0.0 0.0" rpy="0.0 -1.57 0.0" />
-    </collision>
-    <inertial>
-      <mass value="1" />
-      <origin xyz="0.0 0.0 0.0" rpy="0.0 0.0 0.0" />
-      <inertia ixx="1.0" ixy="0.0" ixz="0.0" iyy="1.0" iyz="0.0" izz="1.0"/>
-    </inertial>
-  </link>
-  <joint name="${prefix}ee_fixed_joint" type="fixed">
-    <parent link="${prefix}hook_link" />
-    <child link = "${prefix}ee_link" />
-    <origin xyz="0.0 -0.25 0.0" rpy="0.0 0.0 0.0" />
   </joint>
   <link name="${prefix}ee_link" />
